Commit message: Complete baseline URDF description of Team 10 rover

File: ros2_ws/src/rover_description/urdf/assemblies/mycobot_280_pi_custom.urdf.xacro (robot description, xacro)
@@ -1,4 +1,4 @@
 <?xml version="1.1"?>
-<robot  xmlns:xacro="http://www.ros.org/wiki/xacro" name="mycobot_280_pi_custom" >
+<robot  xmlns:xacro="http://www.ros.org/wiki/xacro" name="mycobot_280_pi_arm" >
 <xacro:macro name="mycobot_280_pi_custom" params="prefix">
 <xacro:property name="width" value=".2" />
@@ -306,3 +306,4 @@
     <mimic joint="${prefix}gripper_controller" multiplier="1.0" offset="0" />
   </joint>
+</xacro:macro>
 </robot>

File: ros2_ws/src/rover_description/urdf/team_10_rover.urdf.xacro (robot description, xacro)
@@ -6,8 +6,8 @@
   <xacro:arg name="arm_xyz" default="0.0880 0 0.0585"/>
   <xacro:arg name="arm_rpy" default="0 0 0"/>
-  <xacro:arg name="lidar_xyz" default="0.0700 0 0.0065"/>
+  <xacro:arg name="lidar_xyz" default="0.0700 0 0.0380"/>
   <xacro:arg name="lidar_rpy" default="0 0 0"/>
-  <xacro:arg name="camera_xyz" default="0 0 0"/>
-  <xacro:arg name="camera_rpy" default="0 0 0"/>
+  <xacro:arg name="camera_xyz" default="0.1746 0 0.0906"/>
+  <xacro:arg name="camera_rpy" default="0 0.4712 0"/>
   <!-- ===================== -->
   <!-- Include LeoRover      -->
@@ -21,8 +21,8 @@
                  mecanum_wheels="$(arg mecanum_wheels)"/>
   <!-- ===================== -->
-  <!-- Include myCobot280    -->
+  <!-- Include myCobot280pi  -->
   <!-- ===================== -->
   <xacro:include filename="$(find rover_description)/urdf/assemblies/mycobot_280_pi_custom.urdf.xacro"/>
-  <xacro:mycobot_280_pi_custom prefix="arm_" >
+  <xacro:mycobot_280_pi_custom prefix="arm_" />
   <!-- ===================== -->
   <!-- Custom Links (Sensors) -->
@@ -31,12 +31,12 @@
     <visual>
       <geometry>
-        <mesh filename="$(find rover_description)/meshes/lidar.stl"/>
+        <mesh filename="package://rover_description/meshes/lidar.stl" scale="0.001 0.001 0.001"/>
       </geometry>
     </visual>
   </link>
-  <link name="camera_link">
+  <link name="depth_camera_link">
     <visual>
       <geometry>
-        <mesh filename="$(find rover_description)/meshes/camera.stl"/>
+        <mesh filename="package://rover_description/meshes/camera.stl" scale="0.001 0.001 0.001"/>
       </geometry>
     </visual>
@@ -58,7 +58,7 @@
   </joint>
   <!-- Attach Camera -->
-  <joint name="camera_joint" type="fixed">
+  <joint name="depth_camera_joint" type="fixed">
     <parent link="base_link"/>
-    <child link="camera_link"/>
+    <child link="depth_camera_link"/>
     <origin xyz="$(arg camera_xyz)" rpy="$(arg camera_rpy)"/>
   </joint>

Commit message: Modify collision boxes for manipulator to exist as simple cylinders, fixing Gazebo physics solver issue.

File: ros2_ws/src/rover_description/urdf/assemblies/mycobot_280_pi_custom.urdf.xacro (robot description, xacro)
@@ -17,7 +17,7 @@
     <collision>
       <geometry>
-       <mesh filename="package://mycobot_description/urdf/mycobot_280_pi/joint1_pi.dae"/>
-      </geometry>
-      <origin xyz="0.0 0 0" rpy="0 0 0"/>
+        <cylinder radius="0.043" length="0.08"/>
+      </geometry>
+      <origin xyz="0.0 0 0.04" rpy="0 0 0"/>
     </collision>
   </link>
@@ -36,7 +36,7 @@
     <collision>
       <geometry>
-       <mesh filename="package://mycobot_description/urdf/mycobot_280_pi/joint2.dae"/>
-      </geometry>
-      <origin xyz="0.0 0 -0.06096" rpy="0 0 -1.5708"/>
+        <cylinder radius="0.024" length="0.084"/>
+      </geometry>
+      <origin xyz="0.0 0 -0.02" rpy="0 0 -1.5708"/>
     </collision>
   </link>
@@ -55,7 +55,7 @@
     <collision>
       <geometry>
-       <mesh filename="package://mycobot_description/urdf/mycobot_280_pi/joint3.dae"/>
-      </geometry>
-      <origin xyz="0.0 0 0.03256" rpy="0 -1.5708 0"/>
+        <cylinder radius="0.024" length="0.150"/>
+      </geometry>
+      <origin xyz="-0.06 0 0.06" rpy="0 -1.5708 0"/>
     </collision>
   </link>
@@ -74,7 +74,7 @@
     <collision>
       <geometry>
-       <mesh filename="package://mycobot_description/urdf/mycobot_280_pi/joint4.dae"/>
-      </geometry>
-      <origin xyz="0.0 0 0.03056" rpy="0 -1.5708 0"/>
+        <cylinder radius="0.024" length="0.135"/>
+      </geometry>
+      <origin xyz="-0.052 0 0.0" rpy="0 -1.5708 0"/>
     </collision>
   </link>
@@ -93,7 +93,7 @@
     <collision>
       <geometry>
-       <mesh filename="package://mycobot_description/urdf/mycobot_280_pi/joint5.dae"/>
-      </geometry>
-      <origin xyz="0.0 -0.001 -0.0345" rpy="0 -1.5708 1.5708"/>
+        <cylinder radius="0.024" length="0.054"/>
+      </geometry>
+      <origin xyz="0.0 0.0 0" rpy="0 1.5708 1.5708"/>
     </collision>
   </link>
@@ -112,7 +112,7 @@
     <collision>
       <geometry>
-       <mesh filename="package://mycobot_description/urdf/mycobot_280_pi/joint6.dae"/>
-      </geometry>
-      <origin xyz="0 0.00 -0.038" rpy="0 0 0"/>
+        <cylinder radius="0.024" length="0.059"/>
+      </geometry>
+      <origin xyz="0 0.00 -0.015" rpy="0 0 0"/>
     </collision>
   </link>
@@ -131,7 +131,7 @@
     <collision>
       <geometry>
-       <mesh filename="package://mycobot_description/urdf/mycobot_280_pi/joint7.dae"/>
-      </geometry>
-      <origin xyz="0.0 0 -0.012" rpy="0 0 0"/>
+        <cylinder radius="0.024" length="0.014"/>
+      </geometry>
+      <origin xyz="0.0 0 -0.007" rpy="0 0 0"/>
     </collision>
   </link>

File: ros2_ws/src/rover_description/urdf/team_10_rover.urdf.xacro (robot description, xacro)
@@ -21,5 +21,5 @@
   <xacro:include filename="$(find leo_description)/urdf/macros.xacro"/>
   <xacro:if value="$(arg use_gazebo)">
-    <xacro:leo_gazebo />
+    <xacro:leo_sim />
   </xacro:if>
   <xacro:unless value="$(arg use_gazebo)">
@@ -42,6 +42,7 @@
     <collision>
       <geometry>
-        <mesh filename="package://rover_description/meshes/lidar.stl" scale="0.001 0.001 0.001"/>
+        <cylinder radius="0.0375" length="0.050"/>
       </geometry>
+      <origin xyz="0 0 -0.025" rpy="0 0 0" />
     </collision>
     <inertial>
@@ -95,6 +96,7 @@
     <collision>
       <geometry>
-        <mesh filename="package://rover_description/meshes/camera.stl" scale="0.001 0.001 0.001"/>
+        <box size="0.09 0.025 0.025" />
       </geometry>
+      <origin xyz="0 0 0" rpy="0 0 -1.5708" />
     </collision>
     <inertial>
