Commit message: Add rover description

File: ros2_ws/src/rover_description/urdf/assemblies/mycobot_280_pi_custom.urdf.xacro (robot description, xacro)
@@ -1,308 +1,377 @@
 <?xml version="1.1"?>
-<robot  xmlns:xacro="http://www.ros.org/wiki/xacro" name="mycobot_280_pi_arm" >
+<robot xmlns:xacro="http://www.ros.org/wiki/xacro" name="mycobot_280_pi_arm">
 <xacro:macro name="mycobot_280_pi_custom" params="prefix">
-<xacro:property name="width" value=".2" />
+  <xacro:property name="width" value=".2" />
   <link name="${prefix}joint1">
-    <visual>
-      <geometry>
-	     <!--- 0.0 0 -0.04  1.5708 3.14159-->
+    <inertial>
+      <origin xyz="0.0 0 0" rpy="0 0 0"/>
+      <mass value="0.20"/>
+      <inertia ixx="0.000105" ixy="0" ixz="0" iyy="0.000105" iyz="0" izz="0.00009"/>
+    </inertial>
+    <visual>
+      <geometry>
        <mesh filename="package://mycobot_description/urdf/mycobot_280_pi/joint1_pi.dae"/>
       </geometry>
-    <origin xyz = "0.0 0 0 " rpy = " 0 0 0"/>
-    </visual>
-    <collision>
-      <geometry>
-	     <!--- 0.0 0 -0.04  1.5708 3.14159-->
-       <mesh filename="package://mycobot_description/urdf/mycobot_280_pi/joint1_pi.dae"/>
-      </geometry>
-    <origin xyz = "0.0 0 0 " rpy = " 0 0 0"/>
+      <origin xyz="0.0 0 0" rpy="0 0 0"/>
+    </visual>
+    <collision>
+      <geometry>
+        <cylinder radius="0.043" length="0.08"/>
+      </geometry>
+      <origin xyz="0.0 0 0.04" rpy="0 0 0"/>
     </collision>
   </link>
   <link name="${prefix}joint2">
+    <inertial>
+      <origin xyz="0.0 0 -0.06096" rpy="0 0 -1.5708"/>
+      <mass value="0.18"/>
+      <inertia ixx="0.00015" ixy="0" ixz="0" iyy="0.00015" iyz="0" izz="0.00008"/>
+    </inertial>
     <visual>
       <geometry>
        <mesh filename="package://mycobot_description/urdf/mycobot_280_pi/joint2.dae"/>
       </geometry>
-    <origin xyz = "0.0 0 -0.06096 " rpy = " 0 0 -1.5708"/>
-    </visual>
-      <collision>
-      <geometry>
-       <mesh filename="package://mycobot_description/urdf/mycobot_280_pi/joint2.dae"/>
-      </geometry>
-    <origin xyz = "0.0 0 -0.06096 " rpy = " 0 0 -1.5708"/>
+      <origin xyz="0.0 0 -0.06096" rpy="0 0 -1.5708"/>
+    </visual>
+    <collision>
+      <geometry>
+        <cylinder radius="0.024" length="0.084"/>
+      </geometry>
+      <origin xyz="0.0 0 -0.02" rpy="0 0 -1.5708"/>
     </collision>
   </link>
   <link name="${prefix}joint3">
+    <inertial>
+      <origin xyz="0.0 0 0.03256" rpy="0 -1.5708 0"/>
+      <mass value="0.15"/>
+      <inertia ixx="0.0001" ixy="0" ixz="0" iyy="0.0001" iyz="0" izz="0.00005"/>
+    </inertial>
     <visual>
       <geometry>
        <mesh filename="package://mycobot_description/urdf/mycobot_280_pi/joint3.dae"/>
       </geometry>
-    <origin xyz = "0.0 0 0.03256 " rpy = " 0 -1.5708 0"/>
-    </visual>
-      <collision>
-        <geometry>
-       <mesh filename="package://mycobot_description/urdf/mycobot_280_pi/joint3.dae"/>
-      </geometry>
-    <origin xyz = "0.0 0 0.03256 " rpy = " 0 -1.5708 0"/>
+      <origin xyz="0.0 0 0.03256" rpy="0 -1.5708 0"/>
+    </visual>
+    <collision>
+      <geometry>
+        <cylinder radius="0.024" length="0.150"/>
+      </geometry>
+      <origin xyz="-0.06 0 0.06" rpy="0 -1.5708 0"/>
     </collision>
   </link>
   <link name="${prefix}joint4">
-    <visual>
-      <geometry>
-       <!--- 0.0 0 -0.04 -->
+    <inertial>
+      <origin xyz="0.0 0 0.03056" rpy="0 -1.5708 0"/>
+      <mass value="0.10"/>
+      <inertia ixx="0.00005" ixy="0" ixz="0" iyy="0.00005" iyz="0" izz="0.00003"/>
+    </inertial>
+    <visual>
+      <geometry>
        <mesh filename="package://mycobot_description/urdf/mycobot_280_pi/joint4.dae"/>
       </geometry>
-    <origin xyz = "0.0 0 0.03056 " rpy = " 0 -1.5708 0"/>
-    </visual>
-      <collision>
-      <geometry>
-       <!--- 0.0 0 -0.04 -->
-       <mesh filename="package://mycobot_description/urdf/mycobot_280_pi/joint4.dae"/>
-      </geometry>
-    <origin xyz = "0.0 0 0.03056 " rpy = " 0 -1.5708 0"/>
-    </collision>
-  </link>
-<link name="${prefix}joint5">
-    <visual>
-      <geometry>
-       <!--- 0.0 0 -0.04 -->
+      <origin xyz="0.0 0 0.03056" rpy="0 -1.5708 0"/>
+    </visual>
+    <collision>
+      <geometry>
+        <cylinder radius="0.024" length="0.135"/>
+      </geometry>
+      <origin xyz="-0.052 0 0.0" rpy="0 -1.5708 0"/>
+    </collision>
+  </link>
+  <link name="${prefix}joint5">
+    <inertial>
+      <origin xyz="0.0 -0.001 -0.0345" rpy="0 -1.5708 1.5708"/>
+      <mass value="0.08"/>
+      <inertia ixx="0.00004" ixy="0" ixz="0" iyy="0.00004" iyz="0" izz="0.00002"/>
+    </inertial>
+    <visual>
+      <geometry>
        <mesh filename="package://mycobot_description/urdf/mycobot_280_pi/joint5.dae"/>
       </geometry>
-    <origin xyz = "0.0 -0.001 -0.0345 " rpy = " 0 -1.5708 1.5708"/>
-    </visual>
-      <collision>
-      <geometry>
-       <!--- 0.0 0 -0.04 -->
-       <mesh filename="package://mycobot_description/urdf/mycobot_280_pi/joint5.dae"/>
-      </geometry>
-    <origin xyz = "0.0 -0.001 -0.0345 " rpy = " 0 -1.5708 1.5708"/>
+      <origin xyz="0.0 -0.001 -0.0345" rpy="0 -1.5708 1.5708"/>
+    </visual>
+    <collision>
+      <geometry>
+        <cylinder radius="0.024" length="0.054"/>
+      </geometry>
+      <origin xyz="0.0 0.0 0" rpy="0 1.5708 1.5708"/>
     </collision>
   </link>
   <link name="${prefix}joint6">
-    <visual>
-      <geometry>
-       <!--- 0.0 0 -0.04 -->
+    <inertial>
+      <origin xyz="0 0.00 -0.038" rpy="0 0 0"/>
+      <mass value="0.05"/>
+      <inertia ixx="0.00002" ixy="0" ixz="0" iyy="0.00002" iyz="0" izz="0.00001"/>
+    </inertial>
+    <visual>
+      <geometry>
        <mesh filename="package://mycobot_description/urdf/mycobot_280_pi/joint6.dae"/>
       </geometry>
-    <origin xyz = "0 0.00 -0.038 " rpy = " 0 0 0"/>
-    </visual>
-      <collision>
-      <geometry>
-       <!--- 0.0 0 -0.04 -->
-       <mesh filename="package://mycobot_description/urdf/mycobot_280_pi/joint6.dae"/>
-      </geometry>
-    <origin xyz = "0 0.00 -0.038 " rpy = " 0 0 0"/>
+      <origin xyz="0 0.00 -0.038" rpy="0 0 0"/>
+    </visual>
+    <collision>
+      <geometry>
+        <cylinder radius="0.024" length="0.059"/>
+      </geometry>
+      <origin xyz="0 0.00 -0.015" rpy="0 0 0"/>
     </collision>
   </link>
   <link name="${prefix}joint6_flange">
-    <visual>
-      <geometry>
-       <!--- 0.0 0 -0.04 -->
+    <inertial>
+      <origin xyz="0.0 0 -0.012" rpy="0 0 0"/>
+      <mass value="0.02"/>
+      <inertia ixx="0.000005" ixy="0" ixz="0" iyy="0.000005" iyz="0" izz="0.000005"/>
+    </inertial>
+    <visual>
+      <geometry>
        <mesh filename="package://mycobot_description/urdf/mycobot_280_pi/joint7.dae"/>
       </geometry>
-    <origin xyz = "0.0 0 -0.012 " rpy = " 0 0 0"/>
-    </visual>
-      <collision>
-      <geometry>
-       <!--- 0.0 0 -0.04 -->
-       <mesh filename="package://mycobot_description/urdf/mycobot_280_pi/joint7.dae"/>
-      </geometry>
-    <origin xyz = "0.0 0 -0.012 " rpy = " 0 0 0"/>
+      <origin xyz="0.0 0 -0.012" rpy="0 0 0"/>
+    </visual>
+    <collision>
+      <geometry>
+        <cylinder radius="0.024" length="0.014"/>
+      </geometry>
+      <origin xyz="0.0 0 -0.007" rpy="0 0 0"/>
+    </collision>
+  </link>
+  <link name="${prefix}gripper_base">
+    <inertial>
+      <origin xyz="0.0 0 -0.012" rpy="0 0 0"/>
+      <mass value="0.07"/>
+      <inertia ixx="0.00002" ixy="0" ixz="0" iyy="0.00002" iyz="0" izz="0.00002"/>
+    </inertial>
+    <visual>
+      <geometry>
+       <mesh filename="package://mycobot_description/urdf/adaptive_gripper/gripper_base.dae"/>
+      </geometry>
+      <origin xyz="0.0 0 -0.012" rpy="0 0 0"/>
+    </visual>
+    <collision>
+      <geometry>
+       <mesh filename="package://mycobot_description/urdf/adaptive_gripper/gripper_base.dae"/>
+      </geometry>
+      <origin xyz="0.0 0 -0.012" rpy="0 0 0"/>
+    </collision>
+  </link>
+  <link name="${prefix}gripper_left1">
+    <inertial>
+      <origin xyz="0 0 0" rpy="0 0 0"/>
+      <mass value="0.005"/>
+      <inertia ixx="0.000001" ixy="0" ixz="0" iyy="0.000001" iyz="0" izz="0.000001"/>
+    </inertial>
+    <visual>
+      <geometry>
+       <mesh filename="package://mycobot_description/urdf/adaptive_gripper/gripper_left1.dae"/>
+      </geometry>
+      <origin xyz="0.039 -0.0133 -0.012" rpy="0 0 0"/>
+    </visual>
+    <collision>
+      <geometry>
+       <mesh filename="package://mycobot_description/urdf/adaptive_gripper/gripper_left1.dae"/>
+      </geometry>
+      <origin xyz="0.039 -0.0133 -0.012" rpy="0 0 0"/>
+    </collision>
+  </link>
+  <link name="${prefix}gripper_left2">
+    <inertial>
+      <origin xyz="0 0 0" rpy="0 0 0"/>
+      <mass value="0.005"/>
+      <inertia ixx="0.000001" ixy="0" ixz="0" iyy="0.000001" iyz="0" izz="0.000001"/>
+    </inertial>
+    <visual>
+      <geometry>
+       <mesh filename="package://mycobot_description/urdf/adaptive_gripper/gripper_left2.dae"/>
+      </geometry>
+      <origin xyz="0.005 -0.0195 -0.012" rpy="0 0 0"/>
+    </visual>
+    <collision>
+      <geometry>
+       <mesh filename="package://mycobot_description/urdf/adaptive_gripper/gripper_left2.dae"/>
+      </geometry>
+      <origin xyz="0.005 -0.0195 -0.012" rpy="0 0 0"/>
+    </collision>
+  </link>
+  <link name="${prefix}gripper_left3">
+    <inertial>
+      <origin xyz="0 0 0" rpy="0 0 0"/>
+      <mass value="0.005"/>
+      <inertia ixx="0.000001" ixy="0" ixz="0" iyy="0.000001" iyz="0" izz="0.000001"/>
+    </inertial>
+    <visual>
+      <geometry>
+       <mesh filename="package://mycobot_description/urdf/adaptive_gripper/gripper_left3.dae"/>
+      </geometry>
+      <origin xyz="0.012 0.0025 -0.012" rpy="0 0 0"/>
+    </visual>
+    <collision>
+      <geometry>
+       <mesh filename="package://mycobot_description/urdf/adaptive_gripper/gripper_left3.dae"/>
+      </geometry>
+      <origin xyz="0.012 0.0025 -0.012" rpy="0 0 0"/>
+    </collision>
+  </link>
+  <link name="${prefix}gripper_right1">
+    <inertial>
+      <origin xyz="0 0 0" rpy="0 0 0"/>
+      <mass value="0.005"/>
+      <inertia ixx="0.000001" ixy="0" ixz="0" iyy="0.000001" iyz="0" izz="0.000001"/>
+    </inertial>
+    <visual>
+      <geometry>
+       <mesh filename="package://mycobot_description/urdf/adaptive_gripper/gripper_right1.dae"/>
+      </geometry>
+      <origin xyz="-0.039 -0.0133 -0.012" rpy="0 0 0"/>
+    </visual>
+    <collision>
+      <geometry>
+       <mesh filename="package://mycobot_description/urdf/adaptive_gripper/gripper_right1.dae"/>
+      </geometry>
+      <origin xyz="-0.039 -0.0133 -0.012" rpy="0 0 0"/>
+    </collision>
+  </link>
+  <link name="${prefix}gripper_right2">
+    <inertial>
+      <origin xyz="0 0 0" rpy="0 0 0"/>
+      <mass value="0.005"/>
+      <inertia ixx="0.000001" ixy="0" ixz="0" iyy="0.000001" iyz="0" izz="0.000001"/>
+    </inertial>
+    <visual>
+      <geometry>
+       <mesh filename="package://mycobot_description/urdf/adaptive_gripper/gripper_right2.dae"/>
+      </geometry>
+      <origin xyz="-0.005 -0.0195 -0.012" rpy="0 0 0"/>
+    </visual>
+    <collision>
+      <geometry>
+       <mesh filename="package://mycobot_description/urdf/adaptive_gripper/gripper_right2.dae"/>
+      </geometry>
+      <origin xyz="-0.005 -0.0195 -0.012" rpy="0 0 0"/>
+    </collision>
+  </link>
+  <link name="${prefix}gripper_right3">
+    <inertial>
+      <origin xyz="0 0 0" rpy="0 0 0"/>
+      <mass value="0.005"/>
+      <inertia ixx="0.000001" ixy="0" ixz="0" iyy="0.000001" iyz="0" izz="0.000001"/>
+    </inertial>
+    <visual>
+      <geometry>
+       <mesh filename="package://mycobot_description/urdf/adaptive_gripper/gripper_right3.dae"/>
+      </geometry>
+      <origin xyz="-0.012 0.0025 -0.012" rpy="0 0 0"/>
+    </visual>
+    <collision>
+      <geometry>
+       <mesh filename="package://mycobot_description/urdf/adaptive_gripper/gripper_right3.dae"/>
+      </geometry>
+      <origin xyz="-0.012 0.0025 -0.012" rpy="0 0 0"/>
     </collision>
   </link>
   <joint name="${prefix}joint2_to_joint1" type="revolute">
     <axis xyz="0 0 1"/>
-    <limit effort = "1000.0" lower = "-2.9321" upper = "2.9321" velocity = "0"/>
+    <limit effort="1000.0" lower="-2.9321" upper="2.9321" velocity="0"/>
     <parent link="${prefix}joint1"/>
     <child link="${prefix}joint2"/>
-    <origin xyz= "0 0 0.13956" rpy = "0 0 0"/>
+    <origin xyz="0 0 0.13956" rpy="0 0 0"/>
+    <dynamics damping="1.0" friction="1.0"/>
   </joint>
   <joint name="${prefix}joint3_to_joint2" type="revolute">
     <axis xyz="0 0 1"/>
-    <limit effort = "1000.0" lower = "-2.4434" upper = "2.4434" velocity = "0"/>
+    <limit effort="1000.0" lower="-2.4434" upper="2.4434" velocity="0"/>
     <parent link="${prefix}joint2"/>
     <child link="${prefix}joint3"/>
-    <origin xyz= "0 0 -0.001" rpy = "0 1.5708 -1.5708"/>
+    <origin xyz="0 0 -0.001" rpy="0 1.5708 -1.5708"/>
+    <dynamics damping="1.0" friction="1.0"/>
   </joint>
   <joint name="${prefix}joint4_to_joint3" type="revolute">
-    <axis xyz=" 0 0 1"/>
-    <limit effort = "1000.0" lower = "-2.6179" upper = "2.6179" velocity = "0"/>
+    <axis xyz="0 0 1"/>
+    <limit effort="1000.0" lower="-2.6179" upper="2.6179" velocity="0"/>
     <parent link="${prefix}joint3"/>
     <child link="${prefix}joint4"/>
-    <origin xyz= "  -0.1104 0 0   " rpy = "0 0 0"/>
+    <origin xyz="-0.1104 0 0" rpy="0 0 0"/>
+    <dynamics damping="1.0" friction="1.0"/>
   </joint>
   <joint name="${prefix}joint5_to_joint4" type="revolute">
-    <axis xyz=" 0 0 1"/>
-    <limit effort = "1000.0" lower = "-2.6179" upper = "2.6179" velocity = "0"/>
+    <axis xyz="0 0 1"/>
+    <limit effort="1000.0" lower="-2.6179" upper="2.6179" velocity="0"/>
     <parent link="${prefix}joint4"/>
     <child link="${prefix}joint5"/>
-    <origin xyz= "-0.096 0 0.06462" rpy = "0 0 -1.5708"/>
+    <origin xyz="-0.096 0 0.06462" rpy="0 0 -1.5708"/>
+    <dynamics damping="1.0" friction="1.0"/>
   </joint>
   <joint name="${prefix}joint6_to_joint5" type="revolute">
     <axis xyz="0 0 1"/>
-    <limit effort = "1000.0" lower = "-2.7052" upper = "2.7925" velocity = "0"/>
+    <limit effort="1000.0" lower="-2.7052" upper="2.7925" velocity="0"/>
     <parent link="${prefix}joint5"/>
     <child link="${prefix}joint6"/>
-    <origin xyz= "0 -0.07318 -0.001" rpy = "1.5708 -1.5708 0"/>
+    <origin xyz="0 -0.07318 -0.001" rpy="1.5708 -1.5708 0"/>
+    <dynamics damping="1.0" friction="1.0"/>
   </joint>
   <joint name="${prefix}joint6output_to_joint6" type="revolute">
     <axis xyz="0 0 1"/>
-    <limit effort = "1000.0" lower = "-3.14159" upper = "3.14159" velocity = "0"/>
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
File: ros2_ws/src/rover_description/urdf/team_10_rover.urdf.xacro (robot description, xacro)
@@ -4,4 +4,5 @@
   <!-- Arguments / Parameters -->
   <!-- ===================== -->
+  <xacro:arg name="use_gazebo" default="false"/>
   <xacro:arg name="arm_xyz" default="0.0880 0 0.0585"/>
   <xacro:arg name="arm_rpy" default="0 0 0"/>
@@ -10,14 +11,15 @@
   <xacro:arg name="camera_xyz" default="0.1746 0 0.0906"/>
   <xacro:arg name="camera_rpy" default="0 0.4712 0"/>
+  <xacro:arg name="robot_ns" default=""/>
   <!-- ===================== -->
   <!-- Include LeoRover      -->
   <!-- ===================== -->
-  <xacro:arg name="fixed" default="false"/>
-  <xacro:arg name="robot_ns" default=""/>
-  <xacro:arg name="mecanum_wheels" default="false"/>
   <xacro:include filename="$(find leo_description)/urdf/macros.xacro"/>
-  <xacro:leo_sim robot_ns="$(arg robot_ns)"
-                 fixed="$(arg fixed)"
-                 mecanum_wheels="$(arg mecanum_wheels)"/>
+  <xacro:if value="$(arg use_gazebo)">
+    <xacro:leo_sim />
+  </xacro:if>
+  <xacro:unless value="$(arg use_gazebo)">
+    <xacro:leo />
+  </xacro:unless>
   <!-- ===================== -->
   <!-- Include myCobot280pi  -->
@@ -34,5 +36,54 @@
       </geometry>
     </visual>
+    <collision>
+      <geometry>
+        <cylinder radius="0.0375" length="0.050"/>
+      </geometry>
+      <origin xyz="0 0 -0.025" rpy="0 0 0" />
+    </collision>
+    <inertial>
+      <mass value="0.190"/>
+      <inertia ixx="0.000095" ixy="0" ixz="0"
+               iyy="0.000095" iyz="0"
+               izz="0.000137"/>
+    </inertial>
   </link>
+<!-- Conditionally boot the Gazebo plugin for lidar -->
+  <xacro:if value="$(arg use_gazebo)">
+    <gazebo reference="lidar_link">
+      <sensor name="rplidar_a2m12" type="gpu_lidar">
+        <always_on>true</always_on>
+        <visualize>true</visualize>
+        <update_rate>10.0</update_rate>
+        <topic>scan</topic>
+        <gz_frame_id>lidar_link</gz_frame_id>
+        <ray>
+          <scan>
+            <horizontal>
+              <samples>1600</samples>
+              <resolution>1</resolution>
+              <min_angle>-3.14159265</min_angle>
+              <max_angle>3.14159265</max_angle>
+            </horizontal>
+            <vertical>
+              <samples>1</samples>
+              <resolution>0.01</resolution>
+              <min_angle>0</min_angle>
+              <max_angle>0</max_angle>
+            </vertical>
+          </scan>
+          <range>
+            <min>0.20</min>
+            <max>12.0</max>
+            <resolution>0.001</resolution> </range>
+          <noise>
+            <type>gaussian</type>
+            <mean>0.0</mean>
+            <stddev>0.01</stddev>
+          </noise>
+        </ray>
+      </sensor>
+    </gazebo>
+  </xacro:if>
   <link name="depth_camera_link">
     <visual>
@@ -41,5 +92,45 @@
       </geometry>
     </visual>
+    <collision>
+      <geometry>
+        <box size="0.09 0.025 0.025" />
+      </geometry>
+      <origin xyz="0 0 0" rpy="0 0 -1.5708" />
+    </collision>
+    <inertial>
+      <mass value="0.072"/>
+      <inertia ixx="0.000052" ixy="0" ixz="0" iyy="0.000007" iyz="0" izz="0.000052"/>
+    </inertial>
   </link>
+  <!-- Required since camera frame is different axis to the model geometry -->
+  <link name="depth_camera_optical_frame"/>
+<!-- Conditionally boot the Gazebo plugin for a depth camera -->
+  <xacro:if value="$(arg use_gazebo)">
+    <gazebo reference="depth_camera_link">
+      <sensor name="depth_camera_sensor" type="rgbd_camera">
+        <always_on>true</always_on>
+        <visualize>true</visualize>
+        <update_rate>30.0</update_rate>
+        <topic>depth_camera</topic>
+        <gz_frame_id>depth_camera_optical_frame</gz_frame_id>
+        <camera name="d435i">
+          <horizontal_fov>1.204</horizontal_fov>
+          <image>
+            <width>1280</width>
+            <height>720</height>
+            <format>R8G8B8</format>
+          </image>
+          <clip>
+            <near>0.28</near>
+            <far>10.0</far>
+          </clip>
+          <noise>
+            <type>gaussian</type>
+            <mean>0.0</mean>
+            <stddev>0.007</stddev> </noise>
+        </camera>
+      </sensor>
+    </gazebo>
+  </xacro:if>
   <!-- ===================== -->
   <!-- Fixed Joints          -->
@@ -63,3 +154,9 @@
     <origin xyz="$(arg camera_xyz)" rpy="$(arg camera_rpy)"/>
   </joint>
+  <!-- & associated optical frame -->
+  <joint name="depth_camera_optical_joint" type="fixed">
+    <parent link="depth_camera_link"/>
+    <child link="depth_camera_optical_frame"/>
+    <origin xyz="0 0 0" rpy="-1.5708 0 -1.5708"/>
+  </joint>
 </robot>
