Commit message: Swap depth bridges to visual bridges rather that topic bridges. Comment and cleanup launch files for sims

File: ros2_ws/src/rover_description/urdf/team_10_rover.urdf.xacro (robot description, xacro)
@@ -11,12 +11,8 @@
   <xacro:arg name="camera_xyz" default="0.1746 0 0.0906"/>
   <xacro:arg name="camera_rpy" default="0 0.4712 0"/>
+  <xacro:arg name="robot_ns" default=""/>
   <!-- ===================== -->
   <!-- Include LeoRover      -->
   <!-- ===================== -->
-<!--
-  <xacro:arg name="fixed" default="false"/>
-  <xacro:arg name="robot_ns" default=""/>
-  <xacro:arg name="mecanum_wheels" default="false"/>
--->
   <xacro:include filename="$(find leo_description)/urdf/macros.xacro"/>
   <xacro:if value="$(arg use_gazebo)">
@@ -53,4 +49,5 @@
     </inertial>
   </link>
+<!-- Conditionally boot the Gazebo plugin for lidar -->
   <xacro:if value="$(arg use_gazebo)">
     <gazebo reference="lidar_link">
@@ -105,12 +102,15 @@
     </inertial>
   </link>
+  <!-- Required since camera frame is different axis to the model geometry -->
+  <link name="depth_camera_optical_frame"/>
+<!-- Conditionally boot the Gazebo plugin for a depth camera -->
   <xacro:if value="$(arg use_gazebo)">
     <gazebo reference="depth_camera_link">
-      <sensor name="camera_sensor" type="rgbd_camera">
+      <sensor name="depth_camera_sensor" type="rgbd_camera">
         <always_on>true</always_on>
         <visualize>true</visualize>
         <update_rate>30.0</update_rate>
-        <topic>camera</topic>
-        <gz_frame_id>depth_camera_link</gz_frame_id>
+        <topic>depth_camera</topic>
+        <gz_frame_id>depth_camera_optical_frame</gz_frame_id>
         <camera name="d435i">
           <horizontal_fov>1.204</horizontal_fov>
@@ -153,3 +153,9 @@
     <origin xyz="$(arg camera_xyz)" rpy="$(arg camera_rpy)"/>
   </joint>
+  <!-- & associated optical frame -->
+  <joint name="depth_camera_optical_joint" type="fixed">
+    <parent link="depth_camera_link"/>
+    <child link="depth_camera_optical_frame"/>
+    <origin xyz="0 0 0" rpy="-1.5708 0 -1.5708"/>
+  </joint>
 </robot>

Commit message: Add optional arm arg for sim speedup

File: ros2_ws/src/rover_description/urdf/team_10_rover.urdf.xacro (robot description, xacro)
@@ -5,4 +5,5 @@
   <!-- ===================== -->
   <xacro:arg name="use_gazebo" default="false"/>
+  <xacro:arg name="use_arm" default="true"/>
   <xacro:arg name="arm_xyz" default="0.0880 0 0.0585"/>
   <xacro:arg name="arm_rpy" default="0 0 0"/>
@@ -37,6 +38,8 @@
   <!-- Include myCobot280pi  -->
   <!-- ===================== -->
-  <xacro:include filename="$(find rover_description)/urdf/assemblies/mycobot_280_pi_custom.urdf.xacro"/>
-  <xacro:mycobot_280_pi_custom prefix="arm_" />
+  <xacro:if value="$(arg use_arm)">
+    <xacro:include filename="$(find rover_description)/urdf/assemblies/mycobot_280_pi_custom.urdf.xacro"/>
+    <xacro:mycobot_280_pi_custom prefix="arm_" />
+  </xacro:if>
   <!-- ===================== -->
   <!-- Custom Links (Sensors) -->
@@ -149,9 +152,11 @@
   <!-- ===================== -->
   <!-- Attach manipulator to LeoRover -->
-  <joint name="arm_mount_joint" type="fixed">
-    <parent link="base_link"/>
-    <child link="arm_joint1"/>
-    <origin xyz="$(arg arm_xyz)" rpy="$(arg arm_rpy)"/>
-  </joint>
+  <xacro:if value="$(arg use_arm)">
+    <joint name="arm_mount_joint" type="fixed">
+      <parent link="base_link"/>
+      <child link="arm_joint1"/>
+      <origin xyz="$(arg arm_xyz)" rpy="$(arg arm_rpy)"/>
+    </joint>
+  </xacro:if>
   <!-- Attach LIDAR -->
   <joint name="lidar_joint" type="fixed">

Commit message: Remove some unnecessary bridges for faster sim

File: ros2_ws/src/rover_description/urdf/team_10_rover.urdf.xacro (robot description, xacro)
@@ -1,4 +1,4 @@
 <?xml version="1.0"?>
-<robot name="team_10_robot" xmlns:xacro="http://www.ros.org/wiki/xacro">
+<robot xmlns:xacro="http://www.ros.org/wiki/xacro" name="team_10_robot">
   <!-- ===================== -->
   <!-- Arguments / Parameters -->
@@ -18,14 +18,12 @@
   <xacro:include filename="$(find leo_description)/urdf/macros.xacro"/>
   <xacro:if value="$(arg use_gazebo)">
-    <xacro:leo_sim />
+    <xacro:leo_sim/>
   </xacro:if>
   <xacro:unless value="$(arg use_gazebo)">
-    <xacro:leo />
+    <xacro:leo/>
   </xacro:unless>
   <xacro:if value="$(arg use_gazebo)">
     <gazebo>
-      <plugin
-        filename="libgz-sim-pose-publisher-system.so"
-        name="gz::sim::systems::PosePublisher">
+      <plugin filename="libgz-sim-pose-publisher-system.so" name="gz::sim::systems::PosePublisher">
         <publish_link_pose>false</publish_link_pose>
         <publish_model_pose>true</publish_model_pose>
@@ -40,5 +38,5 @@
   <xacro:if value="$(arg use_arm)">
     <xacro:include filename="$(find rover_description)/urdf/assemblies/mycobot_280_pi_custom.urdf.xacro"/>
-    <xacro:mycobot_280_pi_custom prefix="arm_" />
+    <xacro:mycobot_280_pi_custom prefix="arm_"/>
   </xacro:if>
   <!-- ===================== -->
@@ -55,14 +53,12 @@
         <cylinder radius="0.0375" length="0.050"/>
       </geometry>
-      <origin xyz="0 0 -0.025" rpy="0 0 0" />
+      <origin xyz="0 0 -0.025" rpy="0 0 0"/>
     </collision>
     <inertial>
       <mass value="0.190"/>
-      <inertia ixx="0.000095" ixy="0" ixz="0"
-               iyy="0.000095" iyz="0"
-               izz="0.000137"/>
+      <inertia ixx="0.000095" ixy="0" ixz="0" iyy="0.000095" iyz="0" izz="0.000137"/>
     </inertial>
   </link>
-<!-- Conditionally boot the Gazebo plugin for lidar -->
+  <!-- Conditionally boot the Gazebo plugin for lidar -->
   <xacro:if value="$(arg use_gazebo)">
     <gazebo reference="lidar_link">
@@ -91,5 +87,6 @@
             <min>0.20</min>
             <max>12.0</max>
-            <resolution>0.001</resolution> </range>
+            <resolution>0.001</resolution>
+          </range>
           <noise>
             <type>gaussian</type>
@@ -109,7 +106,7 @@
     <collision>
       <geometry>
-        <box size="0.09 0.025 0.025" />
+        <box size="0.09 0.025 0.025"/>
       </geometry>
-      <origin xyz="0 0 0" rpy="0 0 -1.5708" />
+      <origin xyz="0 0 0" rpy="0 0 -1.5708"/>
     </collision>
     <inertial>
@@ -120,5 +117,5 @@
   <!-- Required since camera frame is different axis to the model geometry -->
   <link name="depth_camera_optical_frame"/>
-<!-- Conditionally boot the Gazebo plugin for a depth camera -->
+  <!-- Conditionally boot the Gazebo plugin for a depth camera -->
   <xacro:if value="$(arg use_gazebo)">
     <gazebo reference="depth_camera_link">
@@ -126,5 +123,5 @@
         <always_on>true</always_on>
         <visualize>false</visualize>
-        <update_rate>30.0</update_rate>
+        <update_rate>10.0</update_rate>
         <topic>depth_camera</topic>
         <gz_frame_id>depth_camera_optical_frame</gz_frame_id>
@@ -143,5 +140,6 @@
             <type>gaussian</type>
             <mean>0.0</mean>
-            <stddev>0.007</stddev> </noise>
+            <stddev>0.007</stddev>
+          </noise>
         </camera>
       </sensor>
